File: ac_switch/ac_switch.sch (EAGLE design)
At the start: 23 parts, among them IC1 TINY85, T1 BC337

Commit message: Power-Board:  * Widerstands-Packages korrigiert  * Power-LED eingefügt
Parts:
- removed C5: 100n, resistor:C-EU025-024X044
- added LED2: GN, led:LED3MM
- added R4: 220R, resistor:R-EU_0207/10
- LED1: value (none) -> GE
- R2, R3: device resistor:R-EU_0204/7 -> resistor:R-EU_0207/10
Connections:
- new net N$6: LED2.A, R4.1
- net GND: now also LED2.C; no longer C5.1
- net VCC: now also R4.2; no longer C5.2
Changed lines of the file:
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@@
 <grid distance="0.1" unitdist="inch" unit="inch" style="lines" multiple="1" display="no" altdistance="0.01" altunitdist="inch" altunit="inch"/>
 <layers>
-<layer number="1" name="Top" color="4" fill="1" visible="no" active="no"/>
-<layer number="16" name="Bottom" color="1" fill="1" visible="no" active="no"/>
-<layer number="17" name="Pads" color="2" fill="1" visible="no" active="no"/>
-<layer number="18" name="Vias" color="2" fill="1" visible="no" active="no"/>
-<layer number="19" name="Unrouted" color="6" fill="1" visible="no" active="no"/>
-<layer number="20" name="Dimension" color="15" fill="1" visible="no" active="no"/>
-<layer number="21" name="tPlace" color="7" fill="1" visible="no" active="no"/>
-<layer number="22" name="bPlace" color="7" fill="1" visible="no" active="no"/>
-<layer number="23" name="tOrigins" color="15" fill="1" visible="no" active="no"/>
-<layer number="24" name="bOrigins" color="15" fill="1" visible="no" active="no"/>
-<layer number="25" name="tNames" color="7" fill="1" visible="no" active="no"/>
-<layer number="26" name="bNames" color="7" fill="1" visible="no" active="no"/>
-<layer number="27" name="tValues" color="7" fill="1" visible="no" active="no"/>
-<layer number="28" name="bValues" color="7" fill="1" visible="no" active="no"/>
+<layer number="1" name="Top" color="4" fill="1" visible="yes" active="no"/>
+<layer number="16" name="Bottom" color="1" fill="1" visible="yes" active="no"/>
+<layer number="17" name="Pads" color="2" fill="1" visible="yes" active="no"/>
+<layer number="18" name="Vias" color="2" fill="1" visible="yes" active="no"/>
+<layer number="19" name="Unrouted" color="6" fill="1" visible="yes" active="no"/>
+<layer number="20" name="Dimension" color="15" fill="1" visible="yes" active="no"/>
+<layer number="21" name="tPlace" color="7" fill="1" visible="yes" active="no"/>
+<layer number="22" name="bPlace" color="7" fill="1" visible="yes" active="no"/>
+<layer number="23" name="tOrigins" color="15" fill="1" visible="yes" active="no"/>
+<layer number="24" name="bOrigins" color="15" fill="1" visible="yes" active="no"/>
+<layer number="25" name="tNames" color="7" fill="1" visible="yes" active="no"/>
+<layer number="26" name="bNames" color="7" fill="1" visible="yes" active="no"/>
+<layer number="27" name="tValues" color="7" fill="1" visible="yes" active="no"/>
+<layer number="28" name="bValues" color="7" fill="1" visible="yes" active="no"/>
 <layer number="29" name="tStop" color="7" fill="3" visible="no" active="no"/>
 <layer number="30" name="bStop" color="7" fill="6" visible="no" active="no"/>
@@
 <layer number="35" name="tGlue" color="7" fill="4" visible="no" active="no"/>
 <layer number="36" name="bGlue" color="7" fill="5" visible="no" active="no"/>
-<layer number="37" name="tTest" color="7" fill="1" visible="no" active="no"/>
-<layer number="38" name="bTest" color="7" fill="1" visible="no" active="no"/>
+<layer number="37" name="tTest" color="7" fill="1" visible="yes" active="no"/>
+<layer number="38" name="bTest" color="7" fill="1" visible="yes" active="no"/>
 <layer number="39" name="tKeepout" color="4" fill="11" visible="no" active="no"/>
 <layer number="40" name="bKeepout" color="1" fill="11" visible="no" active="no"/>
@@
 <layer number="44" name="Drills" color="7" fill="1" visible="no" active="no"/>
 <layer number="45" name="Holes" color="7" fill="1" visible="no" active="no"/>
-<layer number="46" name="Milling" color="3" fill="1" visible="no" active="no"/>
-<layer number="47" name="Measures" color="7" fill="1" visible="no" active="no"/>
-<layer number="48" name="Document" color="7" fill="1" visible="no" active="no"/>
-<layer number="49" name="Reference" color="7" fill="1" visible="no" active="no"/>
-<layer number="51" name="tDocu" color="7" fill="1" visible="no" active="no"/>
-<layer number="52" name="bDocu" color="7" fill="1" visible="no" active="no"/>
+<layer number="46" name="Milling" color="3" fill="1" visible="yes" active="no"/>
+<layer number="47" name="Measures" color="7" fill="1" visible="yes" active="no"/>
+<layer number="48" name="Document" color="7" fill="1" visible="yes" active="no"/>
+<layer number="49" name="Reference" color="7" fill="1" visible="yes" active="no"/>
+<layer number="51" name="tDocu" color="7" fill="1" visible="yes" active="no"/>
+<layer number="52" name="bDocu" color="7" fill="1" visible="yes" active="no"/>
 <layer number="91" name="Nets" color="2" fill="1" visible="yes" active="yes"/>
 <layer number="92" name="Busses" color="1" fill="1" visible="yes" active="yes"/>
@@
 <part name="C3" library="resistor" deviceset="C-EU" device="025-024X044" value="100n"/>
 <part name="R1" library="resistor" deviceset="R-EU_" device="0207/10" value="10K"/>
-<part name="LED1" library="led" deviceset="LED" device="3MM"/>
-<part name="R2" library="resistor" deviceset="R-EU_" device="0204/7" value="220R"/>
+<part name="LED1" library="led" deviceset="LED" device="3MM" value="GE"/>
+<part name="R2" library="resistor" deviceset="R-EU_" device="0207/10" value="220R"/>
 <part name="U$3" library="n39" deviceset="I3C_PORT" device=""/>
 <part name="U$4" library="n39" deviceset="AVR_ISP" device=""/>
@@
 <part name="C4" library="resistor" deviceset="CPOL-EU" device="E3.5-8" value="68µ"/>
 <part name="U$5" library="n39" deviceset="I3C_PORT" device=""/>
-<part name="R3" library="resistor" deviceset="R-EU_" device="0204/7" value="1,5K"/>
+<part name="R3" library="resistor" deviceset="R-EU_" device="0207/10" value="1,5K"/>
 <part name="U$6" library="n39" deviceset="WAGO_734_262" device=""/>
-<part name="C5" library="resistor" deviceset="C-EU" device="025-024X044" value="100n"/>
 <part name="C6" library="resistor" deviceset="C-EU" device="025-024X044" value="100n"/>
-<part name="GND5" library="supply1" deviceset="GND" device=""/>
-<part name="SUPPLY5" library="supply2" deviceset="VCC" device=""/>
 <part name="SUPPLY6" library="supply2" deviceset="VCC" device=""/>
 <part name="GND6" library="supply1" deviceset="GND" device=""/>
+<part name="LED2" library="led" deviceset="LED" device="3MM" value="GN"/>
+<part name="SUPPLY5" library="supply2" deviceset="VCC" device=""/>
+<part name="GND5" library="supply1" deviceset="GND" device=""/>
+<part name="R4" library="resistor" deviceset="R-EU_" device="0207/10" value="220R"/>
 </parts>
 <sheets>
@@
 <instance part="R3" gate="G$1" x="35.56" y="17.78" rot="R180"/>
 <instance part="U$6" gate="G$1" x="132.08" y="22.86" rot="R90"/>
-<instance part="C5" gate="G$1" x="-73.66" y="5.08" rot="R180"/>
 <instance part="C6" gate="G$1" x="-73.66" y="-17.78" rot="R180"/>
-<instance part="GND5" gate="1" x="-73.66" y="0"/>
-<instance part="SUPPLY5" gate="G$1" x="-73.66" y="12.7"/>
 <instance part="SUPPLY6" gate="G$1" x="-73.66" y="-10.16"/>
 <instance part="GND6" gate="1" x="-73.66" y="-22.86"/>
+<instance part="LED2" gate="G$1" x="-88.9" y="-15.24"/>
+<instance part="SUPPLY5" gate="G$1" x="-88.9" y="5.08"/>
+<instance part="GND5" gate="1" x="-88.9" y="-25.4"/>
+<instance part="R4" gate="G$1" x="-88.9" y="-5.08" rot="R90"/>
 </instances>
 <busses>
@@
 </segment>
 <segment>
-<pinref part="C5" gate="G$1" pin="2"/>
-<pinref part="SUPPLY5" gate="G$1" pin="VCC"/>
-</segment>
-<segment>
 <pinref part="C6" gate="G$1" pin="2"/>
 <pinref part="SUPPLY6" gate="G$1" pin="VCC"/>
+</segment>
+<segment>
+<pinref part="SUPPLY5" gate="G$1" pin="VCC"/>
+<pinref part="R4" gate="G$1" pin="2"/>
+<wire x1="-88.9" y1="2.54" x2="-88.9" y2="0" width="0.1524" layer="91"/>
 </segment>
 </net>
@@
 </segment>
 <segment>
-<pinref part="C5" gate="G$1" pin="1"/>
-<pinref part="GND5" gate="1" pin="GND"/>
-</segment>
-<segment>
 <pinref part="GND6" gate="1" pin="GND"/>
 <pinref part="C6" gate="G$1" pin="1"/>
+</segment>
+<segment>
+<pinref part="LED2" gate="G$1" pin="C"/>
+<pinref part="GND5" gate="1" pin="GND"/>
+<wire x1="-88.9" y1="-20.32" x2="-88.9" y2="-22.86" width="0.1524" layer="91"/>
 </segment>
 </net>
@@
 </segment>
 </net>
+<net name="N$6" class="0">
+<segment>
+<pinref part="R4" gate="G$1" pin="1"/>
+<pinref part="LED2" gate="G$1" pin="A"/>
+<wire x1="-88.9" y1="-10.16" x2="-88.9" y2="-12.7" width="0.1524" layer="91"/>
+</segment>
+</net>
